File: ultra96v2_mipi_csi.kicad_pcb (KiCad board)
At the start: 2 copper layers, 85 x 54 mm, 42 parts, among them J1 61083-063402LF, J2 10075024-G01-20ULF, J3 1-1734248-5, J4 1-1734248-5, U1 AP7361C-33E, U2 SN74AVC4T245PW, U3 PCA9306, U4 PCA9306

Commit message: update
Parts:
- J2: footprint Connector_PinHeader_2.00mm:PinHeader_2x20_P2.00mm_Vertical -> Connector_PinSocket_2.00mm:PinSocket_2x20_P2.00mm_Vertical; moved to B.Cu
- U3, U4: value PCA9306 -> PCA9306DCTR; footprint Package_SO:MSOP-8_3x3mm_P0.65mm -> myfootprint:PCA9306DCTR
- moved R12 99.8 mm to (120.8, 123.8)
- moved R5 77.4 mm to (131.0, 124.0)
- moved R10 68.4 mm to (133.5, 117.2), turned to 180 degrees
- moved C11 65.2 mm to (127.5, 133.8), turned to 180 degrees
- moved R15 64.6 mm to (155.8, 121.5)
- moved C5 61.7 mm to (127.5, 126.0), turned to 180 degrees
- moved C12 61.2 mm to (153.0, 133.5), turned to 180 degrees
- moved C10 58.5 mm to (148.0, 126.0), turned to 180 degrees
- moved C9 56.7 mm to (151.2, 126.0), turned to 180 degrees
- moved R20 54.7 mm to (143.8, 122.0)
- moved C8 54.5 mm to (124.0, 126.0), turned to 180 degrees
- moved R19 53.4 mm to (143.8, 123.8)
- moved R13 51.8 mm to (120.7, 122.0)
- moved R11 51.0 mm to (120.8, 125.5)
- moved C6 46.9 mm to (145.5, 115.2), turned to 90 degrees
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Connections:
- J1 pad 56: Net-(J1-Pad56) -> /HS_CSI1_CLK_N
- J3 pad 5: /HS_CSI0_D1_P -> /HS_CSI0_D1_N
- J4 pad 5: /HS_CSI1_D1_P -> /HS_CSI1_D1_N
- U1 pad 2: Net-(U1-Pad2) -> GND
Routing:
- net GND: track 0.00 -> 306.9 mm, vias 0 -> 90
- net +3V3: track 0.00 -> 132.9 mm, vias 0 -> 8
- net +1V8: track 0.00 -> 92.0 mm, vias 0 -> 4
- net /HS_CSI0_MCLK: track 0.00 -> 53.7 mm, vias 0 -> 2
- net /HS_CSI1_MCLK: track 0.00 -> 52.3 mm, vias 0 -> 1
- net /HS_I2C3_SCL: track 0.00 -> 42.2 mm, vias 0 -> 1
- net /HS_I2C3_SDA: track 0.00 -> 42.0 mm, vias 0 -> 1
- net /CAM0_GPIO: track 0.00 -> 33.2 mm, vias 0 -> 2
- net /CAM1_GPIO: track 0.00 -> 32.9 mm, vias 0 -> 2
- net /CAM0_CLK: track 0.00 -> 29.0 mm, vias 0 -> 2
- net /CAM1_CLK: track 0.00 -> 23.9 mm, vias 0 -> 4
- net /HS_I2C2_SDA: track 0.00 -> 22.2 mm, vias 0 -> 3
- net /HS_I2C2_SCL: track 0.00 -> 20.4 mm, vias 0 -> 3
- net /LS_GPIO_0: track 0.00 -> 17.5 mm, vias 0 -> 1
- net /HS_CSI0_D1_N: track 0.00 -> 17.1 mm, vias 0 -> 1
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- added copper zone on B.Cu, net GND
- added copper zone on F.Cu, net GND
Other:
- board size 85 x 54 mm -> 60 x 45 mm
- board text added: "96-MIPI-CSI Rev.1 (C) Ryuji Fuchikami"

Commit message: この内容で発注
Parts:
- added R21: <0>, Resistor_SMD:R_0603_1608Metric, F.Cu at (120.2, 110.0)
- added R22: <0>, Resistor_SMD:R_0603_1608Metric, F.Cu at (120.2, 111.8)
- moved R4 3.29 mm to (117.0, 111.8)
- moved R3 3.25 mm to (117.0, 110.0)
Connections:
- R4 pad 2: GND -> +1V8
Routing:
- net GND: track 306.9 -> 313.2 mm, vias 90 -> 89
- net +1V8: track 92.0 -> 97.9 mm
- net Net-(R21-Pad1): track 3.85 -> 9.54 mm
- net Net-(R22-Pad1): track 3.08 -> 7.25 mm
- net /LS_GPIO_1: track 16.2 -> 17.7 mm
- net /LS_GPIO_0: track 17.5 -> 18.7 mm

Commit message: rev2
Parts:
- added TP1: TestPoint, TestPoint:TestPoint_THTPad_D1.0mm_Drill0.5mm, F.Cu at (154.4, 104.0)
- J3, J4: footprint myfootprint:55510-140LF -> myfootprint:55510-140LF_handsolder
- moved C11 1.41 mm to (128.9, 133.6)
- moved C5 1.10 mm to (127.5, 124.9)
- moved C8 1.10 mm to (124.0, 124.9)
- moved R11 1.10 mm to (120.8, 124.4)
- moved R12 1.10 mm to (120.8, 122.7)
- moved R13 1.10 mm to (120.7, 120.9)
- moved R5 1.10 mm to (131.0, 122.9)
- moved R6 1.10 mm to (131.0, 120.9)
- moved U3 1.10 mm to (125.8, 122.2)
- moved C12 1.02 mm to (153.2, 134.5)
- moved C10 0.80 mm to (148.0, 125.2)
- moved C9 0.80 mm to (151.2, 125.2)
- moved R14 0.80 mm to (155.8, 122.5)
- moved R15 0.80 mm to (155.8, 120.7)
- moved R18 0.80 mm to (143.8, 124.7)
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Routing:
- net GND: track 313.2 -> 414.7 mm, vias 89 -> 95
- net /HS_I2C3_SCL: track 42.2 -> 60.2 mm, vias 1 -> 3
- net +3V3: track 132.9 -> 144.2 mm
- net /HS_I2C3_SDA: track 42.0 -> 51.2 mm, vias 1 -> 3
- net /CAM1_CLK: track 23.9 -> 32.0 mm
- net /HS_CSI0_D0_N: track 16.8 -> 24.6 mm
- net /HS_CSI0_CLK_P: track 16.8 -> 10.4 mm
- net /HS_CSI1_D1_P: track 11.4 -> 17.3 mm
- net /HS_CSI1_CLK_P: track 11.4 -> 17.3 mm
- net /CAM1_GPIO: track 32.9 -> 38.6 mm
- net /CAM1_SCL: track 14.6 -> 20.1 mm
- net /CAM1_SDA: track 17.1 -> 22.6 mm
- net /HS_CSI1_D0_P: track 11.3 -> 16.6 mm
- net /CAM0_SCL: track 11.6 -> 16.7 mm
- net /CAM0_SDA: track 13.1 -> 18.2 mm
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Other:
- board text added: "96-MIPI-CSI Rev.2 (C) Ryuji Fuchikami"
- board text removed: "96-MIPI-CSI Rev.1 (C) Ryuji Fuchikami"
